File: kicadFiles/anticheww.kicad_pcb (KiCad board)
At the start: 2 copper layers, 303.2 x 94.2 mm, 411 parts, among them J1 Conn_ARM_JTAG_SWD_10, J2 PinHeader_01x09, J3 TYPE-C-31-M12_13, Q1 BSS138, SW1 1U LBKSP, SW10 8, SW11 9, SW12 0, SW13 -_, SW14 +=, SW15 2U BKSP, SW16 Del, SW17 TAB_150, SW18 Q, SW19 W, SW2 ESC, SW20 E, SW21 R, SW22 T, SW23 Y, SW24 U, SW25 I, SW26 O, SW27 P, SW28 [{, SW29 ]}, SW3 1, SW30 1U RBKSP, SW31 Home, SW32 STEPPED_CAPS_125, SW33 CAPS_175, SW34 A, SW35 S, SW36 D, SW37 F, SW38 G, SW39 H, SW4 2, SW40 J, SW41 K, SW42 L, SW43 :;, SW44 "', SW45 \|_150, SW46 ENTER_225, SW47 PgUp, SW48 ISO_ENTER, SW49 RSHIFT_175, SW5 3, SW50 LSHIFT_225, SW51 ISO_100, SW52 Z, SW53 X, SW54 C, SW55 V, SW56 B, SW57 N, SW58 M, SW59 <,, SW6 4, SW60 >., SW61 ?/, SW62 RSHIFT_275, SW63 ISO_\_100, SW64 PgDn, SW65 LSHIFT_125, SW66 LCTRL_125, SW67 LGUI_125, SW68 LALT_125, SW69 SPACE_625, SW7 5, SW70 RALT_125, SW71 FN_125, SW72 RGUI_125, SW73 RCTRL_125, SW74 FN_100, SW75 PgDn, SW76 LCTRL_150, SW77 LGUI_100, SW78 LALT_150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

Commit message: Placed switches, connector, mounting holes
Parts:
- removed CB1, CB3, CB7: 100n, Capacitor_SMD:C_0402_1005Metric
- removed CB2: 100nF, Capacitor_SMD:C_0402_1005Metric
- removed CB4, CB8: 4.7uF, Capacitor_SMD:C_0402_1005Metric
- removed CB5: 1uF, Capacitor_SMD:C_0402_1005Metric
- removed CB6: 10n, Capacitor_SMD:C_0402_1005Metric
- removed CR1, CR2, CRGB1, CRGB10, CRGB2, CRGB3, CRGB4, CRGB5, CRGB6, CRGB7, CRGB8, CRGB9: 100n, Capacitor_SMD:C_0805_2012Metric
- removed CR3: 4.7n, Capacitor_SMD:C_0805_2012Metric_Pad1.15x1.40mm_HandSolder
- removed CR4: 10u, Capacitor_SMD:C_0805_2012Metric_Pad1.15x1.40mm_HandSolder
- removed CSH1, CSH2: 4.7nF, Capacitor_SMD:C_0805_2012Metric
- removed CSI1, CSO1: 1u, Capacitor_SMD:C_0805_2012Metric_Pad1.15x1.40mm_HandSolder
- removed D70, DR1, DROT1, DROT2, DROT3, DROT4: 1N4148, acheron_Components:D_SOD-123
- removed DF1: SMF9.0CA, acheron_Components:D_SOD-123
- removed DS1: RB060M-60TR, acheron_Components:D_SOD-123
- removed F1: 1.5A trip PTC, acheron_Components:Fuse_1812_4532
- removed H1: Half Side Hole, acheron_MountingHoles:halfSideHole
- removed J2: PinHeader_01x09, acheron_Connectors:PinHeader_1x09_P2.54mm_Vertical
- removed J3: TYPE-C-31-M12_13, acheron_Connectors:TYPE-C-31-M-12
- removed L1: OSHLogo, acheron_Graphics:osh-logo
- removed L2, L3, L4, L6: Warning, acheron_Graphics:warning_sign_3.6x3.2mm
- removed L5: Acheron Logo, acheron_Logos:acheronLong
- removed L7: Anticheww Label, antichewwGraphics:antichewwLabel
- removed L8: Anticheww Plated Logo, antichewwGraphics:antichewwLogo_67.9x5
- removed LED1, LED10, LED11, LED12, LED13, LED14, LED15, LED16, LED17, LED18, LED19, LED2, LED20, LED21, LED22, LED23, LED24, LED25, LED26, LED27, LED28, LED29, LED3, LED30, LED31, LED32, LED33, LED34, LED35, LED36, LED37, LED38, LED39, LED4, LED40, LED41, LED42, LED43, LED44, LED45, LED46, LED47, LED48, LED49, LED5, LED50, LED51, LED52, LED53, LED54, LED55, LED56, LED57, LED58, LED59, LED6, LED60, LED61, LED62, LED63, LED64, LED65, LED66, LED67, LED68, LED69, LED7, LED70, LED71, LED72, LED73, LED74, LED75, LED76, LED77, LED78, LED79, LED8, LED80, LED81, LED82, LED83, LED84, LED9: LED, acheron_Components:LED_THT_2.54mm
- removed Q1: BSS138, Package_TO_SOT_SMD:SOT-23
- removed QLED1: AO4407A, acheron_Components:SOIC-8
- removed QLED2, QRST1: DTC123J, Package_TO_SOT_SMD:SOT-23
- removed RCC1, RCC2: 5.1k, acheron_Components:R_SMD_1206
- removed RGB1, RGB10, RGB2, RGB3, RGB4, RGB5, RGB6, RGB7, RGB8, RGB9: WS2812B, acheron_Components:LED_WS2812B_5.0x5.0mm_P3.2mm
- removed RGND1: R01, acheron_Components:R_SMD_1206
- removed RL1, RL10, RL11, RL12, RL13, RL14, RL15, RL16, RL17, RL18, RL19, RL2, RL20, RL21, RL22, RL23, RL24, RL25, RL26, RL27, RL28, RL29, RL3, RL30, RL31, RL32, RL33, RL34, RL35, RL36, RL37, RL38, RL39, RL4, RL40, RL41, RL42, RL43, RL44, RL45, RL46, RL47, RL48, RL49, RL5, RL50, RL51, RL52, RL53, RL54, RL55, RL56, RL57, RL58, RL59, RL6, RL60, RL61, RL62, RL63, RL64, RL65, RL66, RL67, RL68, RL69, RL7, RL70, RL71, RL8, RL9: 420R, acheron_Components:R_SMD_1206
- removed RLED1, RLED2, RR1, RR2, RR3, RR4, RS1, RS2: 10k, acheron_Components:R_SMD_1206
- removed RLED3: 100R, acheron_Components:R_SMD_1206
- removed ROT1, ROT2, ROT3, ROT4: EC11E15244G1, acheron_Hardware:ALPS_EC11E
- removed RR5, RSI1, RSO1: 100k, acheron_Components:R_SMD_1206
- removed RRGB1, RRGB10, RRGB2, RRGB3, RRGB4, RRGB5, RRGB6, RRGB7, RRGB8, RRGB9: 5.1R, acheron_Components:R_SMD_1206
- removed RSH1, RSH2: 1M, acheron_Components:R_SMD_1206
- removed SW76: LCTRL_150, acheron_MX_SolderMask:MX150
- removed SW77: LGUI_100, acheron_MX_SolderMask:MX100
- removed SW78: LALT_150, acheron_MX_SolderMask:MX150
- removed SW79: SPACE_700, acheron_MX_SolderMask:MX700R
- removed SW80: RALT_150, acheron_MX_SolderMask:MX150
- removed SW81: RGUI_100, acheron_MX_SolderMask:MX100
- removed SW82: RCTRL_150, acheron_MX_SolderMask:MX150
- removed SWR1: K2-1187SQ-A4SW-06, acheron_Hardware:smdPushBtn
- removed U1: USBLC6-2SC6, acheron_Components:SOT-23-6
- removed U2: STM32F072CCT6, acheron_Components:LQFP-48_7x7mm_P0.5mm
- removed U3: MCP1700-3302E, Package_TO_SOT_SMD:SOT-23
- D1, D10, D11, D12, D13, D14, D15, D16, D17, D18, D19, D2, D20, D21, D22, D23, D24, D25, D26, D27, D28, D29, D3, D30, D31, D32, D33, D34, D35, D36, D37, D38, D39, D4, D40, D41, D42, D43, D44, D45, D46, D47, D48, D49, D5, D50, D51, D52, D53, D54, D55, D56, D57, D58, D59, D6, D60, D61, D62, D63, D64, D65, D66, D67, D68, D69, D7, D8, D9: value 1N4148 -> 1N4148W
- H10, H3, H4, H5, H6, H9: footprint acheron_MountingHoles:MoutingHole_Oval_BackOnly_7mm_5.0x2.5mm -> acheron_MountingHoles:MountingHole_Oval_7mm_5.0x2.5mm_Leafspring
- H2, H7: footprint acheron_MountingHoles:MoutingHole_Oval_BackOnly_7mm_5.0x2.5mm -> acheron_MountingHoles:MountingHole_Oval_7mm_5.0x2.5mm_Leafspring; moved to F.Cu
- H8: footprint acheron_MountingHoles:MoutingHole_Oval_7mm_5.0x2.5mm -> acheron_MountingHoles:MountingHole_Oval_7mm_5.0x2.5mm_Leafspring
- J1: value Conn_ARM_JTAG_SWD_10 -> TYPE-C-31-M12_13; footprint acheron_Connectors:Conn_ARM_JTAG_SWD_10 -> acheron_Connectors:TYPE-C-31-M-12
- SW1: value 1U LBKSP -> ESC
- SW10: value 8 -> 9
- SW11: value 9 -> 0
- SW12: value 0 -> MINUS
- SW13: value -_ -> PLUS
- SW14: value += -> LBKSP
- SW15: value 2U BKSP -> RBKSP; footprint acheron_MX_SolderMask:MX200 -> acheron_MX_SolderMask:MX100
- SW16: value Del -> PGUP
- SW17: value TAB_150 -> 2U_BKSP; footprint acheron_MX_SolderMask:MX150 -> acheron_MX_SolderMask:MX200
- SW18: value Q -> TAB; footprint acheron_MX_SolderMask:MX100 -> acheron_MX_SolderMask:MX150
- SW19: value W -> Q
- SW2: value ESC -> 1
- SW20: value E -> W
- SW21: value R -> E
- SW22: value T -> R
- SW23: value Y -> T
- SW24: value U -> Y
- SW25: value I -> U
- SW26: value O -> I
- SW27: value P -> O
- SW28: value [{ -> P
- SW29: value ]} -> LBRKT
- SW3: value 1 -> 2
- SW30: value 1U RBKSP -> RBRKT
- SW31: value Home -> BKSLSH; footprint acheron_MX_SolderMask:MX100 -> acheron_MX_SolderMask:MX150
- SW32: value STEPPED_CAPS_125 -> PGDN; footprint acheron_MX_SolderMask:MX125 -> acheron_MX_SolderMask:MX100
- SW33: value CAPS_175 -> CAPS
- SW4: value 2 -> 3
- SW43: value :; -> COLON
- SW44: value "' -> QUOTE
- SW45: value \|_150 -> ENTER; footprint acheron_MX_SolderMask:MX150 -> acheron_MX_SolderMask:MX225R
- SW46: value ENTER_225 -> HOME; footprint acheron_MX_SolderMask:MX225 -> acheron_MX_SolderMask:MX100
- SW47: value PgUp -> LSHFT; footprint acheron_MX_SolderMask:MX100 -> acheron_MX_SolderMask:MX225
- SW48: value ISO_ENTER -> STEPPED_CAPS; footprint acheron_MX_SolderMask:MX_ISOEnter_Vertical_LED -> acheron_MX_SolderMask:MX125
- SW49: value RSHIFT_175 -> Z; footprint acheron_MX_SolderMask:MX175 -> acheron_MX_SolderMask:MX100
- SW5: value 3 -> 4
- SW50: value LSHIFT_225 -> X; footprint acheron_MX_SolderMask:MX225 -> acheron_MX_SolderMask:MX100
- SW51: value ISO_100 -> C
- SW52: value Z -> V
- SW53: value X -> B
- SW54: value C -> N
- SW55: value V -> M
- SW56: value B -> COMMA
- SW57: value N -> DOT
- SW58: value M -> 175_RSHFT; footprint acheron_MX_SolderMask:MX100 -> acheron_MX_SolderMask:MX175
- SW59: value <, -> UP
- SW6: value 4 -> 5
- SW60: value >. -> END
- SW61: value ?/ -> SLSH
- SW62: value RSHIFT_275 -> LCTRL; footprint acheron_MX_SolderMask:MX275 -> acheron_MX_SolderMask:MX125
- SW63: value ISO_\_100 -> LGUI; footprint acheron_MX_SolderMask:MX100 -> acheron_MX_SolderMask:MX125
- SW64: value PgDn -> LALT; footprint acheron_MX_SolderMask:MX100 -> acheron_MX_SolderMask:MX125
- SW65: value LSHIFT_125 -> SPC; footprint acheron_MX_SolderMask:MX125 -> acheron_MX_SolderMask:MX625R
- SW66: value LCTRL_125 -> RALT; footprint acheron_MX_SolderMask:MX125 -> acheron_MX_SolderMask:MX100
- SW67: value LGUI_125 -> RGUI; footprint acheron_MX_SolderMask:MX125 -> acheron_MX_SolderMask:MX100
- SW68: value LALT_125 -> RCTRL; footprint acheron_MX_SolderMask:MX125 -> acheron_MX_SolderMask:MX100
- SW69: value SPACE_625 -> LEFT; footprint acheron_MX_SolderMask:MX625R -> acheron_MX_SolderMask:MX100
- SW7: value 5 -> 6
- SW70: value RALT_125 -> DOWN; footprint acheron_MX_SolderMask:MX125 -> acheron_MX_SolderMask:MX100
- SW71: value FN_125 -> RIGHT; footprint acheron_MX_SolderMask:MX125 -> acheron_MX_SolderMask:MX100
- SW72: value RGUI_125 -> LCTRL; footprint acheron_MX_SolderMask:MX125 -> acheron_MX_SolderMask:MX150
- SW73: value RCTRL_125 -> LGUI; footprint acheron_MX_SolderMask:MX125 -> acheron_MX_SolderMask:MX100
- SW74: value FN_100 -> LALT; footprint acheron_MX_SolderMask:MX100 -> acheron_MX_SolderMask:MX150
- SW75: value PgDn -> SPC; footprint acheron_MX_SolderMask:MX100 -> acheron_MX_SolderMask:MX700R
- SW8: value 6 -> 7
- SW9: value 7 -> 8
- moved D59 558.8 mm to (659.4, 254.5), turned to 0 degrees
- moved D58 557.6 mm to (671.1, 251.1), turned to 0 degrees
- moved D57 537.7 mm to (665.3, 251.1), turned to 0 degrees
- moved D56 524.2 mm to (671.1, 247.8), turned to 0 degrees
- moved D55 488.3 mm to (653.6, 247.8), turned to 0 degrees
- moved D54 470.3 mm to (653.6, 251.1), turned to 0 degrees
- moved D30 458.2 mm to (526.6, 134.5), turned to 0 degrees
- moved D53 448.6 mm to (653.6, 257.8), turned to 0 degrees
- moved D52 433.8 mm to (653.6, 254.5), turned to 0 degrees
- moved D69 432.1 mm to (520.0, 196.1), turned to 0 degrees
- moved D51 425.2 mm to (665.3, 247.8), turned to 0 degrees
- moved D29 420.7 mm to (503.2, 134.5), turned to 0 degrees
- moved D28 408.4 mm to (520.7, 134.5), turned to 0 degrees
- moved D45 404.5 mm to (455.7, 252.1), turned to 0 degrees
- moved D50 401.0 mm to (659.4, 247.8), turned to 0 degrees
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Connections:
- net ROT2_S2 renamed Net-(D30-Pad2)
- D1 pad 1: Row1 -> Net-(D1-Pad1)
- D10 pad 1: Row1 -> Net-(D6-Pad1)
- D10 pad 2: Net-(D10-Pad2) -> Net-(D6-Pad2)
- D11 pad 1: Row1 -> Net-(D13-Pad1)
- D11 pad 2: Net-(D11-Pad2) -> Net-(D13-Pad2)
- D12 pad 1: Row1 -> Net-(D14-Pad1)
- D12 pad 2: Net-(D12-Pad2) -> Net-(D14-Pad2)
- D13 pad 1: Row1 -> Net-(D7-Pad1)
- D13 pad 2: Net-(D13-Pad2) -> Net-(D7-Pad2)
- D14 pad 1: Row1 -> Net-(D8-Pad1)
- D14 pad 2: Net-(D14-Pad2) -> Net-(D8-Pad2)
- D15 pad 1: Row1 -> Net-(D15-Pad1)
- D15 pad 2: ROT1_S2 -> Net-(D15-Pad2)
- D16 pad 1: Row2 -> Net-(D16-Pad1)
- D17 pad 1: Row2 -> Net-(D17-Pad1)
- D18 pad 1: Row2 -> Net-(D18-Pad1)
- D19 pad 1: Row2 -> Net-(D19-Pad1)
- D2 pad 1: Row1 -> Net-(D2-Pad1)
- D20 pad 1: Row2 -> Net-(D20-Pad1)
- D21 pad 1: Row2 -> Net-(D21-Pad1)
- D22 pad 1: Row2 -> Net-(D22-Pad1)
- D23 pad 1: Row2 -> Net-(D23-Pad1)
- D24 pad 1: Row2 -> Net-(D24-Pad1)
- D25 pad 1: Row2 -> Net-(D25-Pad1)
- D26 pad 1: Row2 -> Net-(D26-Pad1)
- D27 pad 1: Row2 -> Net-(D27-Pad1)
- D28 pad 1: Row2 -> Net-(D28-Pad1)
- D29 pad 1: Row2 -> Net-(D29-Pad1)
- D3 pad 1: Row1 -> Net-(D9-Pad1)
- D3 pad 2: Net-(D3-Pad2) -> Net-(D9-Pad2)
- D30 pad 1: Row2 -> Net-(D30-Pad1)
- D31 pad 1: Row3 -> Net-(D31-Pad1)
- D32 pad 1: Row3 -> Net-(D32-Pad1)
- D33 pad 1: Row3 -> Net-(D33-Pad1)
- D34 pad 1: Row3 -> Net-(D34-Pad1)
- D35 pad 1: Row3 -> Net-(D35-Pad1)
- D36 pad 1: Row3 -> Net-(D36-Pad1)
- D37 pad 1: Row3 -> Net-(D37-Pad1)
- D38 pad 1: Row3 -> Net-(D38-Pad1)
- D39 pad 1: Row3 -> Net-(D39-Pad1)
- D4 pad 1: Row1 -> Net-(D10-Pad1)
- D4 pad 2: Net-(D4-Pad2) -> Net-(D10-Pad2)
- D40 pad 1: Row3 -> Net-(D40-Pad1)
- D41 pad 1: Row3 -> Net-(D41-Pad1)
- D42 pad 1: Row3 -> Net-(D42-Pad1)
- D43 pad 1: Row3 -> Net-(D43-Pad1)
- D44 pad 1: Row3 -> Net-(D44-Pad1)
- D45 pad 1: Row3 -> Net-(D45-Pad1)
- D45 pad 2: ROT3_S2 -> Net-(D45-Pad2)
- D46 pad 1: Row4 -> Net-(D46-Pad1)
- D47 pad 1: Row4 -> Net-(D47-Pad1)
- D48 pad 1: Row4 -> Net-(D48-Pad1)
- D49 pad 1: Row4 -> Net-(D49-Pad1)
- D5 pad 1: Row1 -> Net-(D3-Pad1)
- D5 pad 2: Net-(D5-Pad2) -> Net-(D3-Pad2)
- D50 pad 1: Row4 -> Net-(D50-Pad1)
- D51 pad 1: Row4 -> Net-(D51-Pad1)
- D52 pad 1: Row4 -> Net-(D52-Pad1)
- D53 pad 1: Row4 -> Net-(D53-Pad1)
- D54 pad 1: Row4 -> Net-(D54-Pad1)
- D55 pad 1: Row4 -> Net-(D55-Pad1)
- D56 pad 1: Row4 -> Net-(D56-Pad1)
- D57 pad 1: Row4 -> Net-(D57-Pad1)
- D58 pad 1: Row4 -> Net-(D58-Pad1)
- D59 pad 1: Row4 -> Net-(D59-Pad1)
- D6 pad 1: Row1 -> Net-(D4-Pad1)
- D6 pad 2: Net-(D6-Pad2) -> Net-(D4-Pad2)
- D60 pad 1: Row4 -> Net-(D60-Pad1)
- D60 pad 2: ROT4_S2 -> Net-(D60-Pad2)
- D61 pad 1: Row5 -> Net-(D61-Pad1)
- D61 pad 2: L1 -> Net-(D61-Pad2)
- D62 pad 1: Row5 -> Net-(D62-Pad1)
- D62 pad 2: L2 -> Net-(D62-Pad2)
- D63 pad 1: Row5 -> Net-(D63-Pad1)
- D63 pad 2: L3 -> Net-(D63-Pad2)
- D64 pad 1: Row5 -> Net-(D64-Pad1)
- D64 pad 2: L5 -> Net-(D64-Pad2)
- D65 pad 1: Row5 -> Net-(D65-Pad1)
- D65 pad 2: L6 -> Net-(D65-Pad2)
- D66 pad 1: Row5 -> Net-(D66-Pad1)
- D66 pad 2: L7 -> Net-(D66-Pad2)
- D67 pad 1: Row5 -> Net-(D67-Pad1)
- D67 pad 2: L8 -> Net-(D67-Pad2)
- D68 pad 1: Row5 -> Net-(D68-Pad1)
- D68 pad 2: L9 -> Net-(D68-Pad2)
- D69 pad 1: Row5 -> Net-(D69-Pad1)
- D7 pad 1: Row1 -> Net-(D11-Pad1)
- D7 pad 2: Net-(D7-Pad2) -> Net-(D11-Pad2)
- D8 pad 1: Row1 -> Net-(D12-Pad1)
- D8 pad 2: Net-(D8-Pad2) -> Net-(D12-Pad2)
- D9 pad 1: Row1 -> Net-(D5-Pad1)
- D9 pad 2: Net-(D9-Pad2) -> Net-(D5-Pad2)
- SW1 pad 1: Col14 -> Net-(SW1-Pad1)
- SW1 pad 2: Net-(D14-Pad2) -> Net-(D1-Pad2)
- SW10 pad 1: Col9 -> Net-(SW10-Pad1)
- SW10 pad 2: Net-(D9-Pad2) -> Net-(D6-Pad2)
- SW11 pad 1: Col10 -> Net-(SW11-Pad1)
- SW11 pad 2: Net-(D10-Pad2) -> Net-(D13-Pad2)
- SW12 pad 1: Col11 -> Net-(SW12-Pad1)
- SW12 pad 2: Net-(D11-Pad2) -> Net-(D14-Pad2)
- SW13 pad 1: Col12 -> Net-(SW13-Pad1)
- SW13 pad 2: Net-(D12-Pad2) -> Net-(D7-Pad2)
- SW14 pad 1: Col13 -> Net-(SW14-Pad1)
- SW14 pad 2: Net-(D13-Pad2) -> Net-(D8-Pad2)
- SW15 pad 1: Col14 -> Net-(SW15-Pad1)
- SW15 pad 2: Net-(D14-Pad2) -> Net-(D15-Pad2)
- SW16 pad 1: Col15 -> Net-(SW17-Pad1)
- SW16 pad 2: ROT1_S2 -> Net-(D16-Pad2)
- SW17 pad 1: Col1 -> Net-(SW15-Pad1)
- SW17 pad 2: Net-(D16-Pad2) -> Net-(D15-Pad2)
- SW18 pad 1: Col2 -> Net-(SW18-Pad1)
- SW19 pad 1: Col3 -> Net-(SW19-Pad1)
- SW2 pad 1: Col1 -> Net-(SW2-Pad1)
- SW2 pad 2: Net-(D1-Pad2) -> Net-(D2-Pad2)
- SW20 pad 1: Col4 -> Net-(SW20-Pad1)
- SW21 pad 1: Col5 -> Net-(SW21-Pad1)
- SW22 pad 1: Col6 -> Net-(SW22-Pad1)
- SW23 pad 1: Col7 -> Net-(SW23-Pad1)
- SW24 pad 1: Col8 -> Net-(SW24-Pad1)
- SW25 pad 1: Col9 -> Net-(SW25-Pad1)
- SW26 pad 1: Col10 -> Net-(SW26-Pad1)
- SW27 pad 1: Col11 -> Net-(SW27-Pad1)
- SW28 pad 1: Col12 -> Net-(SW28-Pad1)
- SW29 pad 1: Col13 -> Net-(SW29-Pad1)
- SW3 pad 1: Col2 -> Net-(SW3-Pad1)
- SW3 pad 2: Net-(D2-Pad2) -> Net-(D9-Pad2)
- SW30 pad 1: Col14 -> Net-(SW30-Pad1)
- SW31 pad 1: Col15 -> Net-(SW31-Pad1)
- SW32 pad 1: Net-(D31-Pad2) -> Net-(SW32-Pad1)
- SW32 pad 2: Col1 -> Net-(D31-Pad2)
- SW33 pad 1: Col1 -> Net-(SW33-Pad1)
- SW33 pad 2: Net-(D31-Pad2) -> Net-(D32-Pad2)
- SW34 pad 1: Col2 -> Net-(SW34-Pad1)
- SW34 pad 2: Net-(D32-Pad2) -> Net-(D33-Pad2)
- SW35 pad 1: Col3 -> Net-(SW35-Pad1)
- SW35 pad 2: Net-(D33-Pad2) -> Net-(D34-Pad2)
- SW36 pad 1: Col4 -> Net-(SW36-Pad1)
- SW36 pad 2: Net-(D34-Pad2) -> Net-(D35-Pad2)
- SW37 pad 1: Col5 -> Net-(SW37-Pad1)
- SW37 pad 2: Net-(D35-Pad2) -> Net-(D36-Pad2)
- SW38 pad 1: Col6 -> Net-(SW38-Pad1)
- SW38 pad 2: Net-(D36-Pad2) -> Net-(D37-Pad2)
- SW39 pad 1: Col7 -> Net-(SW39-Pad1)
- SW39 pad 2: Net-(D37-Pad2) -> Net-(D38-Pad2)
- SW4 pad 1: Col3 -> Net-(SW4-Pad1)
- SW4 pad 2: Net-(D3-Pad2) -> Net-(D10-Pad2)
- SW40 pad 1: Col8 -> Net-(SW40-Pad1)
- SW40 pad 2: Net-(D38-Pad2) -> Net-(D39-Pad2)
- SW41 pad 1: Col9 -> Net-(SW41-Pad1)
- SW41 pad 2: Net-(D39-Pad2) -> Net-(D40-Pad2)
- SW42 pad 1: Col10 -> Net-(SW42-Pad1)
- SW42 pad 2: Net-(D40-Pad2) -> Net-(D41-Pad2)
- SW43 pad 1: Col11 -> Net-(SW43-Pad1)
- SW43 pad 2: Net-(D41-Pad2) -> Net-(D42-Pad2)
- SW44 pad 1: Col12 -> Net-(SW44-Pad1)
- SW44 pad 2: Net-(D42-Pad2) -> Net-(D43-Pad2)
- SW45 pad 1: Col13 -> Net-(SW45-Pad1)
- SW45 pad 2: Net-(D43-Pad2) -> Net-(D44-Pad2)
- SW46 pad 1: Col14 -> Net-(SW46-Pad1)
- SW46 pad 2: Net-(D44-Pad2) -> Net-(D45-Pad2)
- SW47 pad 1: Col15 -> Net-(SW47-Pad1)
- SW47 pad 2: ROT3_S2 -> Net-(D46-Pad2)
- SW48 pad 1: Col14 -> Net-(SW33-Pad1)
- SW48 pad 2: Net-(D44-Pad2) -> Net-(D32-Pad2)
- SW49 pad 1: Col13 -> Net-(SW49-Pad1)
- SW49 pad 2: Net-(D58-Pad2) -> Net-(D47-Pad2)
- SW5 pad 1: Col4 -> Net-(SW5-Pad1)
- SW5 pad 2: Net-(D4-Pad2) -> Net-(D3-Pad2)
- SW50 pad 1: Col1 -> Net-(SW50-Pad1)
- SW50 pad 2: Net-(D46-Pad2) -> Net-(D48-Pad2)
- SW51 pad 1: Col2 -> Net-(SW51-Pad1)
- SW51 pad 2: Net-(D47-Pad2) -> Net-(D49-Pad2)
- SW52 pad 1: Col3 -> Net-(SW52-Pad1)
- SW52 pad 2: Net-(D48-Pad2) -> Net-(D50-Pad2)
- SW53 pad 1: Col4 -> Net-(SW53-Pad1)
- SW53 pad 2: Net-(D49-Pad2) -> Net-(D51-Pad2)
- SW54 pad 1: Col5 -> Net-(SW54-Pad1)
- SW54 pad 2: Net-(D50-Pad2) -> Net-(D52-Pad2)
- SW55 pad 1: Col6 -> Net-(SW55-Pad1)
- SW55 pad 2: Net-(D51-Pad2) -> Net-(D53-Pad2)
- SW56 pad 1: Col7 -> Net-(SW56-Pad1)
- SW56 pad 2: Net-(D52-Pad2) -> Net-(D54-Pad2)
- SW57 pad 1: Col8 -> Net-(SW57-Pad1)
- SW57 pad 2: Net-(D53-Pad2) -> Net-(D55-Pad2)
- SW58 pad 1: Col9 -> Net-(SW58-Pad1)
- SW58 pad 2: Net-(D54-Pad2) -> Net-(D56-Pad2)
- SW59 pad 1: Col10 -> Net-(SW59-Pad1)
- SW59 pad 2: Net-(D55-Pad2) -> Net-(D57-Pad2)
- SW6 pad 1: Col5 -> Net-(SW6-Pad1)
- SW6 pad 2: Net-(D5-Pad2) -> Net-(D4-Pad2)
- SW60 pad 1: Col11 -> Net-(SW60-Pad1)
- SW60 pad 2: Net-(D56-Pad2) -> Net-(D58-Pad2)
- SW61 pad 1: Col12 -> Net-(SW61-Pad1)
- SW61 pad 2: Net-(D57-Pad2) -> Net-(D59-Pad2)
- SW62 pad 1: Col13 -> Net-(SW62-Pad1)
- SW62 pad 2: Net-(D58-Pad2) -> Net-(D60-Pad2)
- SW63 pad 1: Col14 -> Net-(SW63-Pad1)
- SW63 pad 2: Net-(D59-Pad2) -> Net-(D61-Pad2)
- SW64 pad 1: Col15 -> Net-(SW64-Pad1)
- SW64 pad 2: ROT4_S2 -> Net-(D62-Pad2)
- SW65 pad 1: Col1 -> Net-(SW65-Pad1)
- SW65 pad 2: Net-(D46-Pad2) -> Net-(D63-Pad2)
- SW66 pad 1: Col1 -> Net-(SW66-Pad1)
- SW66 pad 2: L1 -> Net-(D64-Pad2)
- SW67 pad 1: Col2 -> Net-(SW67-Pad1)
- SW67 pad 2: L2 -> Net-(D65-Pad2)
- SW68 pad 1: Col3 -> Net-(SW68-Pad1)
- SW68 pad 2: L3 -> Net-(D66-Pad2)
- SW69 pad 1: Col7 -> Net-(SW69-Pad1)
- SW69 pad 2: L5 -> Net-(D67-Pad2)
- SW7 pad 1: Col6 -> Net-(SW7-Pad1)
- SW7 pad 2: Net-(D6-Pad2) -> Net-(D11-Pad2)
- SW70 pad 1: Col10 -> Net-(SW70-Pad1)
- SW70 pad 2: L6 -> Net-(D68-Pad2)
- SW71 pad 1: Col11 -> Net-(SW71-Pad1)
- SW71 pad 2: L7 -> Net-(D69-Pad2)
- SW72 pad 1: Col12 -> Net-(SW72-Pad1)
- SW72 pad 2: L8 -> Net-(SW72-Pad2)
- SW73 pad 1: Col13 -> Net-(SW73-Pad1)
- SW73 pad 2: L9 -> Net-(SW73-Pad2)
- SW74 pad 1: Col14 -> Net-(SW74-Pad1)
- SW74 pad 2: Net-(D69-Pad2) -> Net-(SW74-Pad2)
- SW75 pad 1: Col15 -> Net-(SW75-Pad1)
- SW8 pad 1: Col7 -> Net-(SW8-Pad1)
- SW8 pad 2: Net-(D7-Pad2) -> Net-(D12-Pad2)
- SW9 pad 1: Col8 -> Net-(SW9-Pad1)
- SW9 pad 2: Net-(D8-Pad2) -> Net-(D5-Pad2)
Routing:
- net Net-(QLED1-Pad5): track 1767.7 -> 0.00 mm, vias 2 -> 0
- net 5V: track 622.4 -> 0.00 mm, vias 4 -> 0
- net Col15: track 526.5 -> 0.00 mm
- net 3.3V: track 466.0 -> 0.00 mm, vias 8 -> 0
- net Col14: track 446.5 -> 0.00 mm
- net Row2: track 415.3 -> 0.00 mm, vias 4 -> 0
- net Row4: track 409.2 -> 0.00 mm, vias 4 -> 0
- net Row1: track 408.2 -> 0.00 mm, vias 4 -> 0
- net Col13: track 405.9 -> 0.00 mm
- net Row3: track 389.4 -> 0.00 mm, vias 4 -> 0
- net Row5: track 368.4 -> 0.00 mm, vias 2 -> 0
- net Col10: track 331.7 -> 0.00 mm
- net ENC_A: track 326.3 -> 0.00 mm, vias 2 -> 0
- net Col12: track 326.1 -> 0.00 mm
- net ENC_B: track 325.1 -> 0.00 mm, vias 2 -> 0
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- added copper zone on F.Cu, net (none)
- removed copper zone on B.Cu, net /SHIELD
- removed copper zone on B.Cu, net 3.3V
- removed copper zone on B.Cu, net GND
- removed copper zone on F.Cu, net GND
- removed copper zone on F.Cu, net GNDD
Other:
- outline, holes or cut-outs redrawn
- board text removed: "(D) 1.25U FN"
- board text removed: "(D) 1.25U RALT"
- board text removed: "(D) 1.25U RCTRL"
- board text removed: "(D) 1.25U RGUI"
- board text removed: "(H) 1.00U RGUI"
- board text removed: "(H,T) 1.50U RCTRL"
- board text removed: "(I) If you want to check or reroute a specific trace, it is recommended that you use the High Contrast mode. Turn it on at View > Contrast mode > Check "High Contrast Mode". The icon is also available at the left icon column."
- board text removed: "(II) It is recommended that the user has some knowledge in Git usage, since it is the main VCS tool used for the Acheron Project."
- board text removed: "(III) All footprints are available either through KiCad's native libraries or the Acheron Library (http://github.com/Gondolindrim/AcheronLibrary). To facilitate the portability of the Acheron projects, this library is generally added at the ${KIPRJMOD} folder as a Git submodule. Hence, right after cloning the PCB repository, run: $ git submodule init --update To update the submodules."
- board text removed: "(IV) For detailed information, check the Acheron Docs page for the ArcticPCB: http://gondolindrim.github.io/AcheronDocs/tsuki/intro.html"
- board text removed: "(T) 1.50U LALT"
- board text removed: "(T) 1.50U LCTRL"
- board text removed: "(T) 1U LGUI"
- board text removed: "(i) The grid unit (1U) value used was 3/4" = 19.05mm"
- board text removed: "(ii) The PCB was designed to fit the standards of the PCBWay manufacturer, at their cheapest settings."
- board text removed: "(iii) All parts were quoted on the LCSC supplier (https://lcsc.com)."
- board text removed: "(iv) You can always contact Gondolindrim through:"
- board text removed: "(v) Most manufacturers list minimum character height as 0.8mm, and warn that any words using values below that will be undiscernable or unreadable. I have found that values down to 0.6mm (25 thou) can be used, although at that level a really close look is needed. Indeed, the minimum character height at which characters are easily readable is 0.8mm"
- board text removed: "- Discord: Gondolindrim#9738"
- board text removed: "- E-mail: alvaro.augusto.volpato@gmail.com"
- board text removed: "- Reddit: /u/gondolindrim"
- board text removed: "- TsukiPCB's GitHub page: http://github.com/Gondolindrim/TsukiPCB"
- board text removed: "1.25U LALT"
- board text removed: "1.25U LCTRL (D)"
- board text removed: "1.25U LGUI (D)"
- board text removed: "1.50U RALT (T)"
- board text removed: "6.0/6.25U STAB"
- board text removed: "6.0/7.0U STAB"
- board text removed: "6.25U"
- board text removed: "6.25U STAB"
- board text removed: "7U STAB"
- board text removed: "7U/6U"
- board text removed: "A10"
- board text removed: "A2"
- board text removed: "A8"
- board text removed: "A9"
- board text removed: "ANSI ENTER"
- board text removed: "Also be sure to check with your parts supplier if they have all the necessary parts in the Bill of Materials and change parts and footprints accordingly to availability"
- board text removed: "B15"
- board text removed: "B3"
- board text removed: "B4"
- board text removed: "B5"
- board text removed: "B6"
- board text removed: "Be aware that capabilities may vary among manufacturers, so be sure to check with your manufacturer if they support the minimum values used."
- board text removed: "GENERAL OBSERVATIONS"
- board text removed: "ISO ENTER"
- board text removed: "ISO ~~#"
- board text removed: "MINIMUM CLEARANCE: 6 thou"
- board text removed: "MINIMUM CLEARANCE: 8 thou"
- board text removed: "MINIMUM VALUES"
- board text removed: "RECOMMENDED VALUES"
- board text removed: "SILKSCREEN CHARACTER HEIGHT: 25 thou (see General Observation (v))"
- board text removed: "SILKSCREEN CHARACTER HEIGHT: 32 thou"
- board text removed: "SILKSCREEN CHARACTER TRACE WIDTH: 6 thou"
- board text removed: "SILKSCREEN CHARACTER TRACE WIDTH: 8 thou"
- board text removed: "STEPPED"
- board text removed: "TRACE WIDTH: 10 thou"
- board text removed: "TRACE WIDTH: 6 thou (approx. 0.15 mm)"
- board text removed: "TRACE-TO-EDGE AND VIA-TO-EDGE DISTANCE: 8 thou"
- board text removed: "These are general hints to use this PCB file. They are aimed specially at thoise new to KiCad or ECAD in general and to whoever wishes to use this project."
- board text removed: "These values were the default values used when possible."
- board text removed: "USAGE GUIDE (PLEASE READ)"
- board text removed: "VIA DIAMETER: 20 thou (approx. 0.5mm)"
- board text removed: "VIA DIAMETER: 32 thou (approx. 0.8mm)"
- board text removed: "VIA HOLE SIZE: 12 thou (approx. 0.3mm)"
- board text removed: "VIA HOLE SIZE: 16 thou (approx. 0.4mm)"
- board text removed: "VIA-TO-VIA AND VIA-TO-TRACE CLEARANCE: 6 thou"
- board text removed: "VIA-TO-VIA AND VIA-TO-TRACE CLEARANCE: 8 thou"
