File: kicadFiles/anticheww.kicad_pcb (KiCad board)
At the start: 2 copper layers, 303.2 x 94.2 mm, 388 parts, among them J1 TYPE-C-31-M-12, J2 ARM JTAG, J3 Extra pins, Q1 AO3401A, Q2 DTC123JKAT146, Q3 DTC123JKAT146, SW1 ESC, SW10 9, SW11 0, SW12 MINUS, SW13 PLUS, SW14 LBKSP, SW15 RBKSP, SW16 2U_BKSP, SW17 TAB, SW18 Q, SW19 W, SW2 1, SW20 E, SW21 R, SW22 T, SW23 Y, SW24 U, SW25 I, SW26 O, SW27 P, SW28 LBRKT, SW29 RBRKT, SW3 2, SW30 BKSLSH, SW31 PGUP, SW32 ISO_ENTER, SW33 CAPS, SW34 A, SW35 S, SW36 D, SW37 F, SW38 G, SW39 H, SW4 3, SW40 J, SW41 K, SW42 L, SW43 COLON, SW44 QUOTE, SW45 ENTER, SW46 HOME, SW47 PGDN, SW48 STEPPED_CAPS, SW49 ISO_TILDE, SW5 4, SW50 LSHFT, SW51 ISO_BKLSH, SW52 Z, SW53 X, SW54 C, SW55 V, SW56 B, SW57 N, SW58 M, SW59 COMMA, SW6 5, SW60 DOT, SW61 SLSH, SW62 175_RSHFT, SW63 UP, SW64 END, SW65 ISO_LSHFT, SW66 LCTRL_125, SW67 LGUI_125, SW68 LALT_125, SW69 SPC_625, SW7 6, SW70 LEFT, SW71 DOWN, SW72 RIGHT, SW73 RALT_125, SW74 RGUI_125, SW75 275_SPC, SW76 SPC_125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

Commit message: Changed PCB file to include plate cutouts
Parts:
- J1: value TYPE-C-31-M-12 -> TYPE-C-31-M12_13
