File: kicadFiles/anticheww.kicad_sch (KiCad schematic)
At the start: 436 parts, among them J1 ARM JTAG, J2 TYPE-C-31-M-12, J3 Extra pins, Q1 AO3401A, Q2 DTC123JKAT146, Q3 DTC123JKAT146, SW1 ESC, SW10 9, SW11 0, SW12 MINUS, SW13 PLUS, SW14 LBKSP, SW15 RBKSP, SW16 2U_BKSP, SW17 TAB, SW18 Q, SW19 W, SW2 1, SW20 E, SW21 R, SW22 T, SW23 Y, SW24 U, SW25 I, SW26 O, SW27 P, SW28 LBRKT, SW29 RBRKT, SW3 2, SW30 BKSLSH, SW31 PGUP, SW32 ISO_ENTER, SW33 CAPS, SW34 A, SW35 S, SW36 D, SW37 F, SW38 G, SW39 H, SW4 3, SW40 J, SW41 K, SW42 L, SW43 COLON, SW44 QUOTE, SW45 ENTER, SW46 HOME, SW47 PGDN, SW48 STEPPED_CAPS, SW49 ISO_TILDE, SW5 4, SW50 LSHFT, SW51 ISO_BKLSH, SW52 Z, SW53 X, SW54 C, SW55 V, SW56 B, SW57 N, SW58 M, SW59 COMMA, SW6 5, SW60 DOT, SW61 SLSH, SW62 175_RSHFT, SW63 UP, SW64 END, SW65 ISO_LSHFT, SW66 275_RSHFT, SW67 LCTRL_125, SW68 LGUI_125, SW69 LALT_125, SW7 6, SW70 SPC_625, SW71 RALT_100, SW72 RGUI_100, SW73 RCTRL_100, SW74 LEFT, SW75 DOWN, SW76 RIGHT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

Commit message: Add requried changes
- Remove encoders support
- Remove 7U and non-blocker bottom row options
- Remove 2.75 right shift option
- Remove mounting holes
- Previous MCU pins used for encoders are now exposed as EXTRA11 and 12
Parts:
- removed C1, C2: 100n, Capacitor_SMD:C_0805_2012Metric, symbol Device:C_Small
- removed D1, D2, D3, D4, D85: 1N4148W, acheron_Components:D_SOD-123, symbol Device:D
- removed FB1: CBG201209U121T, Inductor_SMD:L_0805_2012Metric, symbol Device:Ferrite_Bead_Small
- removed GR4: Warning Sign (7U Space), acheron_Graphics:warning_sign_3.6x3.2mm, symbol Mechanical:MountingHole
- removed GR6: Anticheww Plated Logo, antichewwGraphics:antichewwLogo_67.9x5, symbol Mechanical:MountingHole
- removed GR7: Anticheww Plated Label, antichewwGraphics:antichewwLabel_75x2mm, symbol Mechanical:MountingHole
- removed GR8: Anticheww Plated Label, antichewwGraphics:antichewwLabel_60.9x1.9mm, symbol Mechanical:MountingHole
- removed H1: Mounting Hole, acheron_MountingHoles:MountingHole_Oval_7mm_5.0x2.5mm_Leafspring, symbol Mechanical:MountingHole_Pad
- removed H2, H3, H4, H5, H6, H7, H8, H9: Oval Mounting Hole, acheron_MountingHoles:MountingHole_Oval_7mm_5.0x2.5mm_Leafspring, symbol Mechanical:MountingHole
- removed LED49, LED67, LED69, LED71, LED75, LED80, LED81, LED82, LED89: LED, acheron_Components:LED_THT_2.54mm, symbol acheronSymbols:LED
- removed R1: 10k, acheron_Components:R_0805_2012Metric_LEDs, symbol Device:R
- removed R2, R3, R4: 10k, Resistor_SMD:R_0805_2012Metric, symbol Device:R
- removed R90: 420R, acheron_Components:R_0805_2012Metric_LEDs, symbol Device:R
- removed ROT1, ROT2, ROT3, ROT4: EC11E1820402, acheron_Hardware:ALPS_EC11E, symbol acheronSymbols:Rotary_Encoder_Switch_Chassis
- removed SW66: 275_RSHFT, acheron_MX_SolderMask:MX275, symbol acheronSymbols:MXSwitch
- removed SW71: RALT_100, acheron_MX_SolderMask:MX100, symbol acheronSymbols:MXSwitch
- removed SW72: RGUI_100, acheron_MX_SolderMask:MX100, symbol acheronSymbols:MXSwitch
- removed SW73: RCTRL_100, acheron_MX_SolderMask:MX100, symbol acheronSymbols:MXSwitch
- removed SW77: LCTRL_150, acheron_MX_SolderMask:MX150, symbol acheronSymbols:MXSwitch
- removed SW78: LGUI_100, acheron_MX_SolderMask:MX100, symbol acheronSymbols:MXSwitch
- removed SW79: LALT_150, acheron_MX_SolderMask:MX150, symbol acheronSymbols:MXSwitch
- removed SW80: SPC_700, acheron_MX_SolderMask:MX700R, symbol acheronSymbols:MXSwitch
- removed SW89: RGUI_150, acheron_MX_SolderMask:MX150, symbol acheronSymbols:MXSwitch
- J3: footprint Connector_PinHeader_1.00mm:PinHeader_2x05_P1.00mm_Vertical -> Connector_PinHeader_1.00mm:PinHeader_2x06_P1.00mm_Vertical; symbol Connector_Generic:Conn_02x05_Odd_Even -> Connector_Generic:Conn_02x06_Odd_Even
- renumbered C3 to C1, C12 to C10, C13 to C11, C14 to C12, C15 to C13, C16 to C14, C17 to C15, C18 to C16, C19 to C17, C20 to C18, C21 to C19, C4 to C2, C22 to C20, C27 to C21, C23 to C22, C24 to C23, C28 to C24, C29 to C25, C30 to C26, C25 to C27, C26 to C28, C5 to C3, C6 to C4, C7 to C5, C8 to C6, C9 to C7, C10 to C8, C11 to C9, D19 to D1, D28 to D10, D29 to D11, D30 to D12, D31 to D13, D32 to D14, D33 to D15, D5 to D16, D6 to D17, D7 to D18, D8 to D19, D20 to D2, D9 to D20, D10 to D21, D11 to D22, D34 to D23, D35 to D24, D36 to D25, D37 to D26, D38 to D27, D39 to D28, D40 to D29, D21 to D3, D41 to D30, D42 to D31, D43 to D32, D44 to D33, D45 to D34, D46 to D35, D47 to D36, D48 to D37, D12 to D38, D13 to D39, D22 to D4, D14 to D40, D15 to D41, D16 to D42, D17 to D43, D18 to D44, D49 to D45, D50 to D46, D51 to D47, D52 to D48, D53 to D49, D23 to D5, D54 to D50, D55 to D51, D56 to D52, D57 to D53, D58 to D54, D59 to D55, D60 to D56, D61 to D57, D62 to D58, D63 to D59, D24 to D6, D64 to D60, D65 to D61, D66 to D62, D67 to D63, D68 to D64, D69 to D65, D70 to D66, D71 to D67, D72 to D68, D73 to D69, D25 to D7, D74 to D70, D75 to D71, D76 to D72, D77 to D73, D78 to D74, D79 to D75, D80 to D76, D81 to D77, D82 to D78, D83 to D79, D26 to D8, D84 to D80, D86 to D81, D87 to D82, D88 to D83, D89 to D84, D90 to D85, D91 to D86, D92 to D87, D27 to D9, FB2 to FB1, GR5 to GR4, J2 to J1, J1 to J2, LED50 to LED49, LED51 to LED50, LED52 to LED51, LED53 to LED52, LED54 to LED53, LED55 to LED54, LED56 to LED55, LED57 to LED56, LED58 to LED57, LED59 to LED58, LED60 to LED59, LED61 to LED60, LED62 to LED61, LED63 to LED62, LED64 to LED63, LED65 to LED64, LED66 to LED65, LED68 to LED66, LED70 to LED67, LED72 to LED68, LED73 to LED69, LED74 to LED70, LED76 to LED71, LED77 to LED72, LED78 to LED73, LED79 to LED74, LED87 to LED75, LED88 to LED76, LED83 to LED77, LED84 to LED78, LED85 to LED79, LED86 to LED80, R5 to R1, R14 to R10, R15 to R11, R16 to R12, R17 to R13, R18 to R14, R95 to R15, R96 to R16, R19 to R17, R20 to R18, R21 to R19, R6 to R2, R22 to R20, R23 to R21, R24 to R22, R25 to R23, R26 to R24, R27 to R25, R28 to R26, R29 to R27, R30 to R28, R31 to R29, R7 to R3, R32 to R30, R33 to R31, R34 to R32, R35 to R33, R36 to R34, R37 to R35, R38 to R36, R39 to R37, R40 to R38, R41 to R39, R8 to R4, R42 to R40, R43 to R41, R44 to R42, R45 to R43, R46 to R44, R47 to R45, R48 to R46, R49 to R47, R50 to R48, R51 to R49, R9 to R5, R97 to R50, R52 to R51, R53 to R52, R54 to R53, R55 to R54, R56 to R55, R57 to R56, R58 to R57, R59 to R58, R60 to R59, R10 to R6, R61 to R60, R62 to R61, R63 to R62, R64 to R63, R65 to R64, R66 to R65, R98 to R66, R99 to R67, R100 to R68, R101 to R69, R11 to R7, R67 to R70, R68 to R71, R69 to R72, R70 to R73, R71 to R74, R72 to R75, R73 to R76, R74 to R77, R75 to R78, R76 to R79, R12 to R8, R77 to R80, R78 to R81, R79 to R82, R80 to R83, R81 to R84, R82 to R85, R83 to R86, R84 to R87, R85 to R88, R86 to R89, R13 to R9, R87 to R90, R88 to R91, R89 to R92, R91 to R93, R92 to R94, R93 to R95, R94 to R96, SW67 to SW66, SW68 to SW67, SW69 to SW68, SW70 to SW69, SW74 to SW70, SW75 to SW71, SW76 to SW72, SW87 to SW73, SW88 to SW74, SW81 to SW75, SW82 to SW76, SW83 to SW77, SW84 to SW78, SW85 to SW79, SW86 to SW80, U3 to U2, U2 to U3
Connections:
- net ROTA renamed EXTRA12
- net EXTRA12: now also J3.12 (Pin_12)
- net ROTB renamed EXTRA11
- net EXTRA11: now also J3.11 (Pin_11)
- net S7: no longer names the net of D79.2 (A), SW73.2 (Row)
- net S8: no longer names the net of D80.2 (A), SW74.2 (Row)
Other:
- note removed: "7.00 blocker (TB)"
- note removed: "700 (T)"
- note removed: "7U (T)"
- note removed: "ENCODERS"
- note removed: "Mounting holes"
- note removed: "No blocker (N)"
